File: kicad/v2/v2.kicad_sch (KiCad schematic)
At the start: 13 parts, among them J1 IN+/IN-, J2 Raspberry_Pi_2_3, J2 TP4056, J3 MT3608, J3 TDA1308, J4 AudioJack3, J5 PCM5102, SW1 SW_SPST, SW2 SW_Push, SW3 SW_Push, SW4 SW_Push, SW5 SW_Push

Commit message: feat: update schematic
Parts:
- added J3: Conn_01x09, Connector_PinHeader_2.54mm:PinHeader_1x09_P2.54mm_Vertical, symbol Connector_Generic:Conn_01x09
- BT1: footprint (none) -> Connector_PinHeader_2.54mm:PinHeader_1x02_P2.54mm_Vertical
- J1: renamed from J2; footprint (none) -> Connector_PinHeader_2.54mm:PinHeader_2x20_P2.54mm_Vertical
- J2: renamed from J3; footprint (none) -> Connector_PinSocket_2.54mm:PinSocket_1x04_P2.54mm_Vertical
- J4: renamed from J5; footprint (none) -> Connector_PinSocket_2.54mm:PinSocket_1x08_P2.54mm_Vertical
- J5: renamed from J2; footprint (none) -> Connector_PinSocket_2.54mm:PinSocket_1x06_P2.54mm_Vertical
- J6: renamed from J3; footprint (none) -> Connector_PinSocket_2.54mm:PinSocket_1x08_P2.54mm_Vertical
- J7: renamed from J4; footprint (none) -> Connector_Audio:Jack_3.5mm_PJ320D_Horizontal
- J8: renamed from J1; footprint (none) -> Connector_PinHeader_2.54mm:PinHeader_1x02_P2.54mm_Vertical
- SW1: renamed from SW2; footprint (none) -> Button_Switch_THT:SW_PUSH_6mm_H5mm
- SW2: renamed from SW3; footprint (none) -> Button_Switch_THT:SW_PUSH_6mm_H5mm
- SW3: renamed from SW4; footprint (none) -> Button_Switch_THT:SW_PUSH_6mm_H5mm
- SW4: renamed from SW5; footprint (none) -> Button_Switch_THT:SW_PUSH_6mm_H5mm
- SW5: renamed from SW1; footprint (none) -> Button_Switch_THT:SW_Slide_SPDT_Straight_CK_OS102011MS2Q
Connections:
- net GND: now also J3.2 (Pin_2)
- net at J1.1 (3V3), J1.17 (3V3): now also J3.1 (Pin_1)
- net at J1.11 (GPIO17): now also J3.7 (Pin_7)
- net at J1.18 (GPIO24): now also J3.8 (Pin_8)
- net at J1.19 (MOSI0/GPIO10): now also J3.3 (Pin_3)
- net at J1.22 (GPIO25): now also J3.6 (Pin_6)
- net at J1.23 (SCLK0/GPIO11): now also J3.4 (Pin_4)
- net at J1.24 (~{CE0}/GPIO8): now also J3.5 (Pin_5)
- net at J1.33 (PWM1/GPIO13): now also J3.9 (Pin_9)
Other:
- moved on the sheet: J5
